Commit message: upgrade for depth camera

File: src/my_robot/urdf/my_robot.xacro (robot description, xacro)
@@ -185,3 +185,10 @@
     <dynamics damping="1.0" friction="1.0"/>
   </joint>
+  <joint name="camera_optical_joint" type="fixed">
+    <origin xyz="0 0 0" rpy="-1.5707 0 -1.5707"/>
+    <parent link="camera"/>
+    <child link="camera_link_optical"/>
+  </joint>
+  <link name="camera_link_optical">
+  </link>
 </robot>

Commit message: finish up project

File: src/my_robot/urdf/my_robot.xacro (robot description, xacro)
@@ -43,8 +43,20 @@
       </geometry>
     </visual>
+    <collision name='front_caster_collision'>
+      <origin xyz="0.20 0 -0.07" rpy=" 0 0 0"/>
+      <geometry>
+        <sphere radius="0.079"/>
+      </geometry>
+    </collision>
+    <visual name='front_caster_visual'>
+      <origin xyz="0.20 0 -0.07" rpy=" 0 0 0"/>
+      <geometry>
+        <sphere radius="0.08"/>
+      </geometry>
+    </visual>
     <collision name='back_caster_collision'>
       <origin xyz="-0.20 0 -0.07" rpy=" 0 0 0"/>
       <geometry>
-        <sphere radius="0.08"/>
+        <sphere radius="0.079"/>
       </geometry>
     </collision>
@@ -106,5 +118,5 @@
   </link>
   <joint type="continuous" name="left_wheel_hinge">
-    <origin xyz="0.15 0.2 0" rpy="0 0 0"/>
+    <origin xyz="0 0.2 0" rpy="0 0 0"/>
     <child link="left_wheel"/>
     <parent link="chassis"/>
@@ -114,5 +126,5 @@
   </joint>
   <joint type="continuous" name="right_wheel_hinge">
-    <origin xyz="0.15 -0.2 0" rpy="0 0 0"/>
+    <origin xyz="0 -0.2 0" rpy="0 0 0"/>
     <child link="right_wheel"/>
     <parent link="chassis"/>
